File: ki_cad/MCU.kicad_sch (KiCad schematic)
At the start: 13 parts, among them J11 SWD_CONN, SW1 USER_SW, U1 STM32L010F4P6

Commit message: update after feedback (purchased)
Parts:
- removed SW1: USER_SW, Custom:SW_PUSH_TS-1088-AR02016, symbol Switch:SW_DPST_x2
- added SW1: USER_SW, Custom:SW_PUSH_TS-1088-AR02016, symbol Switch:SW_Push
- R20, R21: footprint Resistor_SMD:R_0201_0603Metric -> Resistor_SMD:R_0402_1005Metric; JLCPCB Part # C22843 -> C25900
Connections:
- net at R1.2, U1.12 (PA6): now also SW1.2
- net at R2.2: now also SW1.1
Changed lines of the file:
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@@
 	(rectangle
 		(start 121.92 72.39)
-		(end 158.75 99.06)
+		(end 149.86 99.06)
 		(stroke
 			(width 0.0254)
@@
 	(text "Programming Connector"
 		(exclude_from_sim no)
-		(at 139.954 101.092 0)
+		(at 135.89 101.092 0)
 		(effects
 			(font
@@
 	(wire
 		(pts
+			(xy 35.56 64.77) (xy 35.56 63.5)
+		)
+		(stroke
+			(width 0)
+			(type default)
+		)
+	)
+	(wire
+		(pts
 			(xy 129.54 88.9) (xy 134.62 88.9)
 		)
@@
 	(wire
 		(pts
+			(xy 35.56 63.5) (xy 41.91 63.5)
+		)
+		(stroke
+			(width 0)
+			(type default)
+		)
+	)
+	(wire
+		(pts
 			(xy 77.47 86.36) (xy 134.62 86.36)
 		)
@@
 		(pts
 			(xy 144.78 36.83) (xy 148.59 36.83)
-		)
-		(stroke
-			(width 0)
-			(type default)
-		)
-	)
-	(wire
-		(pts
-			(xy 34.29 63.5) (xy 41.91 63.5)
 		)
 		(stroke
@@
 					(size 1.27 1.27)
 				)
-				(justify right)
+				(justify left)
 			)
 		)
@@
 			)
 		)
-		(property "Footprint" "Resistor_SMD:R_0201_0603Metric"
+		(property "Footprint" "Resistor_SMD:R_0402_1005Metric"
 			(at 104.902 71.12 90)
 			(effects
@@
 			)
 		)
-		(property "JLCPCB Part #" "C22843"
+		(property "JLCPCB Part #" "C25900"
 			(at 106.68 71.12 90)
 			(effects
@@
 			)
 		)
-		(property "Footprint" "Resistor_SMD:R_0201_0603Metric"
+		(property "Footprint" "Resistor_SMD:R_0402_1005Metric"
 			(at 97.282 71.12 90)
 			(effects
@@
 			)
 		)
-		(property "JLCPCB Part #" "C22843"
+		(property "JLCPCB Part #" "C25900"
 			(at 99.06 71.12 90)
 			(effects
@@
 	)
 	(symbol
-		(lib_id "Switch:SW_DPST_x2")
+		(lib_id "Switch:SW_Push")
 		(at 154.94 43.18 270)
 		(unit 1)
@@
 		(on_board yes)
 		(dnp no)
-		(fields_autoplaced yes)
 		(property "Reference" "SW1"
-			(at 157.48 41.9099 90)
+			(at 157.734 41.656 90)
 			(effects
 				(font
@@
 		)
 		(property "Value" "USER_SW"
-			(at 157.48 44.4499 90)
+			(at 157.226 44.958 90)
 			(effects
 				(font
@@
 		)
 		(property "Footprint" "Custom:SW_PUSH_TS-1088-AR02016"
-			(at 154.94 43.18 0)
+			(at 160.02 43.18 0)
 			(effects
 				(font
@@
 		)
 		(property "Datasheet" "~"
-			(at 154.94 43.18 0)
-			(effects
-				(font
-					(size 1.27 1.27)
-				)
-				(hide yes)
-			)
-		)
-		(property "Description" "Single Pole Single Throw (SPST) switch, separate symbol"
+			(at 160.02 43.18 0)
+			(effects
+				(font
+					(size 1.27 1.27)
+				)
+				(hide yes)
+			)
+		)
+		(property "Description" "Push button switch, generic, two pins"
 			(at 154.94 43.18 0)
 			(effects
@@
 				(hide yes)
 			)
-		)
-		(property "Field9" ""
-			(at 154.94 43.18 90)
-			(effects
-				(font
-					(size 1.27 1.27)
-				)
-				(hide yes)
-			)
-		)
-		(pin "4"
-		)
-		(pin "3"
 		)
 		(pin "1"
@@
 	(symbol
 		(lib_id "power:GND")
-		(at 34.29 63.5 0)
+		(at 35.56 64.77 0)
 		(unit 1)
 		(exclude_from_sim no)
@@
 		(fields_autoplaced yes)
 		(property "Reference" "#PWR020"
-			(at 34.29 69.85 0)
+			(at 35.56 71.12 0)
 			(effects
 				(font
@@
 		)
 		(property "Value" "GND"
-			(at 34.29 68.58 0)
+			(at 35.56 69.85 0)
 			(effects
 				(font
@@
 		)
 		(property "Footprint" ""
-			(at 34.29 63.5 0)
+			(at 35.56 64.77 0)
 			(effects
 				(font
@@
 		)
 		(property "Datasheet" ""
-			(at 34.29 63.5 0)
+			(at 35.56 64.77 0)
 			(effects
 				(font
@@
 		)
 		(property "Description" "Power symbol creates a global label with name \"GND\" , ground"
-			(at 34.29 63.5 0)
-			(effects
-				(font
+			(at 35.56 64.77 0)
+			(effects
+				(font

Commit message: update parts && add test points
Parts:
- added TP_SCL1, TP_SDA1: TestPoint, TestPoint:TestPoint_Pad_D1.5mm, symbol Connector:TestPoint
- R2, R3, R4: footprint Resistor_SMD:R_0201_0603Metric -> Resistor_SMD:R_0402_1005Metric; JLCPCB Part # C22843 -> C25867
Connections:
- net SCL: now also TP_SCL1.1
- net SDA: now also TP_SDA1.1
Other:
- note added: "SWD DEBUG"
- moved on the sheet: D2, D3, J11, R1, R2, R3, R4, SW1

Commit message: update code
Parts:
- removed R2: 1K5, Resistor_SMD:R_0402_1005Metric, symbol Device:R
Connections:
- net +3V3: now also SW1.1
Changed lines of the file:
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@@
 	)
 	(rectangle
-		(start 144.78 20.32)
+		(start 144.78 30.48)
 		(end 190.5 69.85)
 		(stroke
@@
 	(text "Debug stuff\n(to be deleted in Release)"
 		(exclude_from_sim no)
-		(at 166.624 17.018 0)
+		(at 168.148 27.432 0)
 		(effects
 			(font
@@
 	(no_connect
 		(at 41.91 60.96)
-	)
-	(wire
-		(pts
-			(xy 177.8 27.94) (xy 177.8 29.21)
-		)
-		(stroke
-			(width 0)
-			(type default)
-		)
 	)
 	(wire
@@
 		)
 		(instances
-			(project ""
+			(project "pwm_board"
 				(path "/71ddf0e9-b3bd-413d-a31e-e27757e0e466/7c9a574e-1626-44f3-9594-09b30c5119d2"
 					(reference "SW1")
@@
 		)
 		(instances
-			(project ""
+			(project "pwm_board"
 				(path "/71ddf0e9-b3bd-413d-a31e-e27757e0e466/7c9a574e-1626-44f3-9594-09b30c5119d2"
 					(reference "U1")
@@
 		)
 		(instances
-			(project ""
+			(project "pwm_board"
 				(path "/71ddf0e9-b3bd-413d-a31e-e27757e0e466/7c9a574e-1626-44f3-9594-09b30c5119d2"
 					(reference "TP_SCL1")
@@
 	(symbol
 		(lib_id "power:+3V3")
-		(at 177.8 27.94 0)
+		(at 177.8 36.83 0)
 		(unit 1)
 		(exclude_from_sim no)
@@
 		(dnp no)
 		(property "Reference" "#PWR010"
-			(at 177.8 31.75 0)
+			(at 177.8 40.64 0)
 			(effects
 				(font
@@
 		)
 		(property "Value" "+3V3"
-			(at 177.8 24.13 0)
+			(at 177.8 33.02 0)
 			(effects
 				(font
@@
 		)
 		(property "Footprint" ""
-			(at 177.8 27.94 0)
+			(at 177.8 36.83 0)
 			(effects
 				(font
@@
 		)
 		(property "Datasheet" ""
-			(at 177.8 27.94 0)
+			(at 177.8 36.83 0)
 			(effects
 				(font
@@
 		)
 		(property "Description" "Power symbol creates a global label with name \"+3V3\""
-			(at 177.8 27.94 0)
+			(at 177.8 36.83 0)
 			(effects
 				(font
@@
 		)
 		(instances
-			(project ""
+			(project "pwm_board"
 				(path "/71ddf0e9-b3bd-413d-a31e-e27757e0e466/7c9a574e-1626-44f3-9594-09b30c5119d2"
 					(reference "J11")
 					(unit 1)
 				)
-			)
-		)
-	)
-	(symbol
-		(lib_id "Device:R")
-		(at 177.8 33.02 0)
-		(unit 1)
-		(exclude_from_sim no)
-		(in_bom yes)
-		(on_board yes)
-		(dnp no)
-		(property "Reference" "R2"
-			(at 175.006 33.02 0)
-			(effects
-				(font
-					(size 1.27 1.27)
-				)
-			)
-		)
-		(property "Value" "1K5"
-			(at 181.356 33.02 0)
-			(effects
-				(font
-					(size 1.27 1.27)
-				)
-			)
-		)
-		(property "Footprint" "Resistor_SMD:R_0402_1005Metric"
-			(at 176.022 33.02 90)
-			(effects
-				(font
-					(size 1.27 1.27)
-				)
-				(hide yes)
-			)
-		)
-		(property "Datasheet" "~"
-			(at 177.8 33.02 0)
-			(effects
-				(font
-					(size 1.27 1.27)
-				)
-				(hide yes)
-			)
-		)
-		(property "Description" "Resistor"
-			(at 177.8 33.02 0)
-			(effects
-				(font
-					(size 1.27 1.27)
-				)
-				(hide yes)
-			)
-		)
-		(property "JLCPCB Part #" "C25867"
-			(at 177.8 33.02 90)
-			(effects
-				(font
-					(size 1.27 1.27)
-				)
-				(hide yes)
-			)
-		)
-		(property "KLC_S3.3" ""
-			(at 177.8 33.02 90)
-			(effects
-				(font
-					(size 1.27 1.27)
-				)
-				(hide yes)
-			)
-		)
-		(property "KLC_S4.1" ""
-			(at 177.8 33.02 90)
-			(effects
-				(font
-					(size 1.27 1.27)
-				)
-				(hide yes)
-			)
-		)
-		(property "Sim.Device" ""
-			(at 177.8 33.02 90)
-			(effects
-				(font
-					(size 1.27 1.27)
-				)
-				(hide yes)
-			)
-		)
-		(property "Sim.Type" ""
-			(at 177.8 33.02 90)
-			(effects
-				(font
-					(size 1.27 1.27)
-				)
-				(hide yes)
-			)
-		)
-		(property "Field9" ""
-			(at 177.8 33.02 0)
-			(effects
-				(font
-					(size 1.27 1.27)
-				)
-				(hide yes)
-			)
-		)
-		(pin "2"
-		)
-		(pin "1"
-		)
-		(instances
-			(project "pwm_board"
-				(path "/71ddf0e9-b3bd-413d-a31e-e27757e0e466/7c9a574e-1626-44f3-9594-09b30c5119d2"
-					(reference "R2")
-					(unit 1)
-				)
