File: ki_cad/pwm.kicad_sch (KiCad schematic)
At the start: 52 parts, among them J0 Conn_01x03_Pin, J1 Conn_01x03_Pin, J12 Conn_01x02_Pin, J13 Conn_01x02_Pin, J14 Conn_01x02_Pin, J15 Conn_01x02_Pin, J16 Conn_01x02_Pin, J17 Conn_01x02_Pin, J2 Conn_01x03_Pin, J3 Conn_01x03_Pin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

Commit message: update after feedback (purchased)
Parts:
- removed C13: 10u, Capacitor_SMD:C_0402_1005Metric, symbol Device:C
- removed U4: PCA9685PW, Package_SO:TSSOP-28_4.4x9.7mm_P0.65mm, symbol Driver_LED:PCA9685PW
- added C21: 10u, Capacitor_SMD:C_0402_1005Metric, symbol Device:C
- added U5: PCA9635PW,118, Package_SO:TSSOP-28_4.4x9.7mm_P0.65mm, symbol Driver_LED:PCA9635
- D4, D5, D6, D7, D8, D9: footprint Diode_SMD:D_SOD-523 -> Diode_SMD:D_SOD-323; JLCPCB Part # C146342 -> C5334579
Connections:
- net +3V3: now also C21.2, U5.28 (VDD); no longer J4.2 (Pin_2), J5.2 (Pin_2), J6.2 (Pin_2), J7.2 (Pin_2), J8.2 (Pin_2), J9.2 (Pin_2)
- net GND: now also C21.1, U5.1 (A0), U5.14 (VSS), U5.2 (A1), U5.24 (A5), U5.25 (A6), U5.3 (A2), U5.4 (A3), U5.5 (A4)
- net MOTOR_PWM_0: now also U5.17 (LED10)
- net MOTOR_PWM_1: now also U5.18 (LED11)
- net MOTOR_PWM_2: now also U5.19 (LED12)
- net MOTOR_PWM_3: now also U5.20 (LED13)
- net MOTOR_PWM_4: now also U5.21 (LED14)
- net MOTOR_PWM_5: now also U5.22 (LED15)
- net OE: now also U5.23 (~{OE})
- net SCL: now also U5.26 (SCL)
- net SDA: now also U5.27 (SDA)
- net SERVO_PWM_0: now also U5.6 (LED0)
- net SERVO_PWM_1: now also U5.7 (LED1)
- net SERVO_PWM_2: now also U5.8 (LED2)
- net SERVO_PWM_3: now also U5.9 (LED3)
- net SERVO_PWM_4: now also U5.10 (LED4)
- net SERVO_PWM_5: now also U5.11 (LED5)
- net SERVO_PWM_6: now also U5.12 (LED6)
- net SERVO_PWM_7: now also U5.13 (LED7)
- net SERVO_PWM_8: now also U5.15 (LED8)
- net SERVO_PWM_9: now also U5.16 (LED9)
- new net +3V3_1: J4.2 (Pin_2), J5.2 (Pin_2), J6.2 (Pin_2), J7.2 (Pin_2), J8.2 (Pin_2), J9.2 (Pin_2)
Other:
- note added: "Servos suppled by first Buck-Converter"
- note added: "Servos suppled by second Buck-Converter"
- note added: "Suppled by second Buck-Converter"
- moved on the sheet: C14, C15, C2, C5, C6, C7, D4, D5, D6, D7, D8, D9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
